Commit message: depth cam and imu placed upper case added

File: src/rhex_description/urdf/accessories.xacro (robot description, xacro)
@@ -2,11 +2,33 @@
 <robot xmlns:xacro="http://ros.org/wiki/xacro">
     <xacro:arg name="lidar_enabled" default="true"/>
+    <!-- Define robot constants -->
+    <xacro:property name="base_width" value="0.2"/>
+    <xacro:property name="base_length" value="0.554"/>
+    <xacro:property name="base_height" value="0.112"/>
+    <xacro:property name="upper_case_z_position" value="0.055"/>
+    <xacro:property name="imu_y_position" value="-0.005"/>
+    <xacro:property name="imu_z_position" value="${base_height/2 + 0.031}"/>
+    <xacro:property name="depth_cam_x_position" value="${base_length/2 - 0.0075}"/>
+    <xacro:property name="depth_cam_y_position" value="0.0055"/>
     <!-- IMU (Internal Measurement Unit) -->
     <link name="imu_link">
-        <xacro:box_inertia mass="0.001" width="0.01" height="0.01" length="0.01">
+        <visual>
+            <origin xyz="0 0 0" rpy="0 0 0"/>
+            <geometry>
+                <box size="0.015 0.115 0.020"/>
+            </geometry>
+        </visual>
+        <collision>
+            <origin xyz="0 0 0" rpy="0 0 0"/>
+            <geometry>
+                <box size="0.015 0.115 0.020"/>
+            </geometry>
+        </collision>
+        <xacro:box_inertia mass="0.001" width="0.01" height="0.01" length="0.01"> <!-- Did not take into account of dimensions added later by me-->
             <origin xyz="0 0 0" rpy="0 0 0" />
         </xacro:box_inertia>
     </link>
     <joint name="imu_joint" type="fixed">
+        <origin xyz="${base_length/2} ${imu_y_position} ${imu_z_position}" rpy="0 0 0"/>
         <parent link="base_link" />
         <child link="imu_link" />
@@ -101,5 +123,5 @@
         <parent link="base_link"/>
         <child link="lidar_frame"/>
-        <origin xyz="0 0 ${base_height/2 + 0.025}" rpy="0 0 0"/>
+        <origin xyz="0 0 ${2*upper_case_z_position + base_height/2}" rpy="0 0 0"/>
     </joint>
     <xacro:if value="$(arg lidar_enabled)">
@@ -144,5 +166,5 @@
             <origin xyz="0 0 0" rpy="0 0 0"/>
             <geometry>
-                <box size="0.015 0.13 0.022"/>
+                <box size="0.015 0.0867 0.022"/>
             </geometry>
         </visual>
@@ -150,8 +172,8 @@
             <origin xyz="0 0 0" rpy="0 0 0"/>
             <geometry>
-                <box size="0.015 0.13 0.022"/>
+                <box size="0.015 0.0867 0.022"/>
             </geometry>
         </collision>
-        <xacro:box_inertia mass="0.02" width="0.015" height="0.022" length="0.13">
+        <xacro:box_inertia mass="0.02" width="0.015" height="0.022" length="0.0867">
             <origin xyz="0 0 0" rpy="0 0 0"/>
         </xacro:box_inertia>
@@ -160,5 +182,5 @@
         <parent link="base_link"/>
         <child link="camera_link"/>
-        <origin xyz="${base_length/2} 0 0" rpy="0 0 0"/>
+        <origin xyz="${depth_cam_x_position} ${depth_cam_y_position} ${base_height}" rpy="0 0 0"/>
     </joint>
     <link name="camera_depth_frame"/>

File: src/rhex_description/urdf/robot.urdf.xacro (robot description, xacro)
@@ -5,4 +5,5 @@
     <xacro:property name="base_length" value="0.554"/>
     <xacro:property name="base_height" value="0.112"/>
+    <xacro:property name="upper_case_z_position" value="0.055"/>
     <xacro:property name="ground_clearance" value="0.155"/>
     <xacro:property name="mid_legs_xoff" value="0.0"/>
@@ -41,4 +42,25 @@
         <child link="base_inertia_link"/>
     </joint>
+    <!-- Upper case of the robot added -->
+    <link name="upper_case_link">
+        <visual>
+            <origin xyz="0 0 0" rpy="0 0 0"/>
+            <geometry>
+                <mesh filename="file://$(find rhex_description)/urdf/meshes/upper_case.dae" scale="0.001 0.001 0.001"/>
+            </geometry>
+            <material name="Cyan"/> <!-- Material color added but not working-->
+        </visual>
+        <collision>
+            <origin xyz="0 0 0" rpy="0 0 0"/>
+            <geometry>
+                <mesh filename="file://$(find rhex_description)/urdf/meshes/upper_case.dae" scale="0.001 0.001 0.001"/>
+            </geometry>
+        </collision>
+    </link>
+    <joint name="base_upper_case_joint" type="fixed">
+        <origin xyz="0 0 ${upper_case_z_position}" rpy="0 0 0"/>
+        <parent link="base_link"/>
+        <child link="upper_case_link"/>
+    </joint>
     <!-- Include the rest of the simulation properties and body parts-->
     <xacro:include filename="robot_gazebo.xacro"/>
